File: 4ch-spdt-relay-1fan-arduino-nano-pcb.kicad_pcb (KiCad board)
At the start: 2 copper layers, 147 x 97.2 mm, 54 parts, among them J1 Screw_Terminal_01x03, J2 Conn_01x08_Pin, J3 Screw_Terminal_01x03, J4 Screw_Terminal_01x03, J5 Screw_Terminal_01x03, J7 Conn_01x07_Pin, J9 Conn_01x04_Pin, K1 G5LE-1, K2 G5LE-1, K3 G5LE-1, K4 G5LE-1, Q1 2N3904, Q2 2N3904, Q3 2N3904, Q4 2N3904, Q5 BT136, U5 MOC3021M, U6 PC817, U7 TSOP1738, U8 HLK-10M05

Commit message: Add files via upload
Parts:
- removed the REF** at (76.5, 31.2)
- removed the REF** at (216.4, 31.1)
- removed the REF** at (76.4, 121.2)
- removed the REF** at (216.2, 121.1)
- added REF**: MountingHole_2.5mm_Pad, MountingHole:MountingHole_2.5mm_Pad, F.Cu at (220.8, 148.6)
- added REF**: MountingHole_2.5mm_Pad, MountingHole:MountingHole_2.5mm_Pad, F.Cu at (220.7, 58.4)
- added REF**: MountingHole_2.5mm_Pad, MountingHole:MountingHole_2.5mm_Pad, F.Cu at (83.9, 148.4)
- added REF**: MountingHole_2.5mm_Pad, MountingHole:MountingHole_2.5mm_Pad, F.Cu at (84.0, 58.4)
- moved BR1 28.2 mm to (175.7, 87.9)
- moved J3 28.2 mm to (117.3, 65.2)
- moved J4 28.2 mm to (134.4, 65.1)
- moved A1 28.2 mm to (103.8, 136.7)
- moved D1 28.2 mm to (99.8, 96.2)
- moved D2 28.2 mm to (99.7, 102.4)
- moved D3 28.2 mm to (117.3, 102.4)
- moved D4 28.2 mm to (117.6, 96.2)
- moved D5 28.2 mm to (134.5, 102.4)
- moved D7 28.2 mm to (150.9, 102.4)
- moved D8 28.2 mm to (151.0, 96.2)
- moved J1 28.2 mm to (100.2, 65.1)
- moved J2 28.2 mm to (134.6, 113.6)
- moved J5 28.2 mm to (151.5, 65.1)
- moved J6 28.2 mm to (178.1, 64.4)
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Routing:
- net GND: track 211.1 -> 258.0 mm
- net Net-(J6-Pin_2): track 26.0 -> 62.4 mm
- net +5V: track 239.1 -> 269.3 mm
- net Net-(J6-Pin_1): track 51.9 -> 81.5 mm
Other:
- board size 147 x 97.2 mm -> 143.9 x 97.2 mm
